File: USBFAN-MOTOR-CONTROL/USBFAN-MOTOR-CONTROL.kicad_pcb (KiCad board)
At the start: 0 parts

Commit message: schematics finalized and pcb generated.
 Changes to be committed:
	modified:   USBFAN-MOTOR-CONTROL/USBFAN-MOTOR-CONTROL.kicad_pcb
	modified:   USBFAN-MOTOR-CONTROL/USBFAN-MOTOR-CONTROL.kicad_prl
	modified:   USBFAN-MOTOR-CONTROL/USBFAN-MOTOR-CONTROL.kicad_sch
	new file:   USBFAN-MOTOR-CONTROL/fp-info-cache
Parts:
- added C1: 100n, Capacitor_SMD:C_0603_1608Metric_Pad1.08x0.95mm_HandSolder, B.Cu at (116.7, 76.3)
- added C10: 1uF, Capacitor_SMD:C_0805_2012Metric_Pad1.18x1.45mm_HandSolder, B.Cu at (105.5, 99.5)
- added C2: 470uF16V, Capacitor_THT:CP_Radial_D8.0mm_P3.50mm, F.Cu at (109.3, 68.5)
- added C3: 100n, Capacitor_SMD:C_0603_1608Metric_Pad1.08x0.95mm_HandSolder, B.Cu at (110.6, 70.3)
- added C4: 100n, Capacitor_SMD:C_0603_1608Metric_Pad1.08x0.95mm_HandSolder, B.Cu at (116.8, 63.7)
- added C5: 10uF, Capacitor_SMD:C_0805_2012Metric_Pad1.18x1.45mm_HandSolder, B.Cu at (114.9, 63.5)
- added C6: 100n, Capacitor_SMD:C_0603_1608Metric_Pad1.08x0.95mm_HandSolder, B.Cu at (103.0, 112.5)
- added C7: 470uF16V, Capacitor_THT:CP_Radial_D8.0mm_P3.50mm, F.Cu at (106.8, 89.0)
- added C8: 470uF16V, Capacitor_THT:CP_Radial_D8.0mm_P3.50mm, F.Cu at (110.6, 97.4)
- added C9: 100n, Capacitor_SMD:C_0603_1608Metric_Pad1.08x0.95mm_HandSolder, B.Cu at (113.5, 100.1)
- added D1: 1N5819, Diode_SMD:D_SOD-323_HandSoldering, B.Cu at (109.7, 63.5)
- added D2: 1N5819, Diode_SMD:D_SOD-323_HandSoldering, B.Cu at (115.0, 84.0)
- added D3: 1N5819, Diode_SMD:D_SOD-323_HandSoldering, B.Cu at (112.5, 81.0)
- added D4: 0805,White, LED_SMD:LED_0805_2012Metric_Pad1.15x1.40mm_HandSolder, B.Cu at (104.1, 109.0)
- added F1: Polyfuse, Fuse:Fuse_0805_2012Metric_Pad1.15x1.40mm_HandSolder, B.Cu at (106.7, 63.5)
- added J1: USB_C_2P, pcblib_new599 Library:USB_TYPE_C_2P_THT_90, F.Cu at (112.4, 59.9)
- added J2: Conn_01x20, Connector_PinSocket_2.54mm:PinSocket_1x20_P2.54mm_Vertical, F.Cu at (101.6, 60.0)
- added J3: Conn_01x20, Connector_PinSocket_2.54mm:PinSocket_1x20_P2.54mm_Vertical, F.Cu at (119.4, 108.3)
- added J4: USB_A, Connector_USB:USB_A_CONNFLY_DS1095-WNR0, F.Cu at (107.0, 137.1)
- added L1: L, Inductor_THT:L_Radial_D10.0mm_P5.00mm_Fastron_07M, F.Cu at (109.5, 76.0)
- added Q1: AO3400A, Package_TO_SOT_SMD:SOT-23, B.Cu at (114.3, 89.5)
- added R1: 220, Resistor_SMD:R_0603_1608Metric_Pad0.98x0.95mm_HandSolder, B.Cu at (117.0, 84.0)
- added R2: 7.5K, Resistor_SMD:R_0603_1608Metric_Pad0.98x0.95mm_HandSolder, B.Cu at (117.1, 89.5)
- added R3: 220, Resistor_SMD:R_0603_1608Metric_Pad0.98x0.95mm_HandSolder, B.Cu at (104.1, 105.0)
- added R4: 220, Resistor_SMD:R_0603_1608Metric_Pad0.98x0.95mm_HandSolder, B.Cu at (101.3, 112.5)
- added R5: 7.5K, Resistor_SMD:R_0603_1608Metric_Pad0.98x0.95mm_HandSolder, B.Cu at (114.8, 76.4)
- added RV1: B10K, pcblib_new599 Library:POT_SINGLE_WH148, B.Cu at (110.5, 113.5)
- added SW1: SW_Push, Button_Switch_THT:SW_PUSH_6mm_H7.3mm, B.Cu at (106.8, 109.3)
Other:
- board outline added: 21 x 96 mm
- copper layers 0 -> 2
